Commit message: corrected launch file and version erro

File: arm_bot/description/arm_ros2_control.xacro (robot description, xacro)
@@ -4,5 +4,5 @@
         <xacro:property name="PI" value="3.14159265359" />
             <hardware>
-                <plugin>ign_ros2_control/IgnitionSystem</plugin>
+                <plugin>gz_ros2_control/GazeboSimSystem</plugin>
             </hardware>
         <joint name="Joint_1">

File: arm_bot/description/robot.urdf.xacro (robot description, xacro)
@@ -53,5 +53,5 @@
       <origin rpy="3.14 0 0" xyz="0 0 0.07785"/>
       <geometry>
-        <mesh filename="file:///home/linux/arm_ws/src/arm_bot/meshes/basecone.STL" scale="0.001 0.001 0.001"/>
+        <mesh filename="package://arm_bot/meshes/basecone.STL" scale="0.001 0.001 0.001"/>
       </geometry>
       <material name="">
@@ -62,5 +62,5 @@
       <origin rpy="3.14 0 0" xyz="0 0 0.07785"/>
       <geometry>
-        <mesh filename="file:///home/linux/arm_ws/src/arm_bot/meshes/basecone.STL" scale="0.001 0.001 0.001"/>
+        <mesh filename="package://arm_bot/meshes/basecone.STL" scale="0.001 0.001 0.001"/>
       </geometry>
     </collision>
@@ -76,5 +76,5 @@
       <origin rpy="0 0 0" xyz="0 0 0"/>
       <geometry>
-        <mesh filename="file:///home/linux/arm_ws/src/arm_bot/meshes/body20.STL" scale="0.001 0.001 0.001"/>
+        <mesh filename="package://arm_bot/meshes/body20.STL" scale="0.001 0.001 0.001"/>
       </geometry>
       <material name="">
@@ -85,5 +85,5 @@
       <origin rpy="0 0 0" xyz="0 0 0"/>
       <geometry>
-        <mesh filename="file:///home/linux/arm_ws/src/arm_bot/meshes/body20.STL" scale="0.001 0.001 0.001"/>
+        <mesh filename="package://arm_bot/meshes/body20.STL" scale="0.001 0.001 0.001"/>
       </geometry>
     </collision>
@@ -101,5 +101,5 @@
       <origin rpy="3.14 0 0.785" xyz="0 0 0.0"/>
       <geometry>
-        <mesh filename="file:///home/linux/arm_ws/src/arm_bot/meshes/Ring48_20p.STL" scale="0.001 0.001 0.001"/>
+        <mesh filename="package://arm_bot/meshes/Ring48_20p.STL" scale="0.001 0.001 0.001"/>
       </geometry>
       <material name="">
@@ -110,5 +110,5 @@
       <origin rpy="3.14 0 0.785" xyz="0 0 0.0"/>
       <geometry>
-        <mesh filename="file:///home/linux/arm_ws/src/arm_bot/meshes/Ring48_20p.STL" scale="0.001 0.001 0.001"/>
+        <mesh filename="package://arm_bot/meshes/Ring48_20p.STL" scale="0.001 0.001 0.001"/>
       </geometry>
     </collision>
@@ -124,5 +124,5 @@
       <origin rpy="0 0 3.14" xyz="0.0556 0.0253 0"/>
       <geometry>
-        <mesh filename="file:///home/linux/arm_ws/src/arm_bot/meshes/shoulderplate.STL" scale="0.001 0.001 0.001"/>
+        <mesh filename="package://arm_bot/meshes/shoulderplate.STL" scale="0.001 0.001 0.001"/>
       </geometry>
       <material name="">
@@ -133,5 +133,5 @@
       <origin rpy="0 0 3.14" xyz="0.0556 0.0253 0"/>
       <geometry>
-        <mesh filename="file:///home/linux/arm_ws/src/arm_bot/meshes/shoulderplate.STL" scale="0.001 0.001 0.001"/>
+        <mesh filename="package://arm_bot/meshes/shoulderplate.STL" scale="0.001 0.001 0.001"/>
       </geometry>
     </collision>
@@ -147,5 +147,5 @@
       <origin rpy="-1.5707 0 1.5707" xyz="0 0 0.057"/>
       <geometry>
-        <mesh filename="file:///home/linux/arm_ws/src/arm_bot/meshes/shouldershell.STL" scale="0.001 0.001 0.001"/>
+        <mesh filename="package://arm_bot/meshes/shouldershell.STL" scale="0.001 0.001 0.001"/>
       </geometry>
       <material name="">
@@ -156,5 +156,5 @@
       <origin rpy="-1.5707 0 1.5707" xyz="0 0 0.057"/>
       <geometry>
-        <mesh filename="file:///home/linux/arm_ws/src/arm_bot/meshes/shouldershell.STL" scale="0.001 0.001 0.001"/>
+        <mesh filename="package://arm_bot/meshes/shouldershell.STL" scale="0.001 0.001 0.001"/>
       </geometry>
     </collision>
@@ -170,5 +170,5 @@
       <origin rpy="0 1.5707 0" xyz="-0.062 0 0"/>
       <geometry>
-        <mesh filename="file:///home/linux/arm_ws/src/arm_bot/meshes/shouldercap.STL" scale="0.001 0.001 0.001"/>
+        <mesh filename="package://arm_bot/meshes/shouldercap.STL" scale="0.001 0.001 0.001"/>
       </geometry>
       <material name="">
@@ -179,5 +179,5 @@
       <origin rpy="0 1.5707 0" xyz="-0.062 0 0"/>
       <geometry>
-        <mesh filename="file:///home/linux/arm_ws/src/arm_bot/meshes/shouldercap.STL" scale="0.001 0.001 0.001"/>
+        <mesh filename="package://arm_bot/meshes/shouldercap.STL" scale="0.001 0.001 0.001"/>
       </geometry>
     </collision>
@@ -193,5 +193,5 @@
       <origin rpy="0 1.5707 0" xyz="0.005 0 0"/>
       <geometry>
-        <mesh filename="file:///home/linux/arm_ws/src/arm_bot/meshes/body20.STL" scale="0.001 0.001 0.001"/>
+        <mesh filename="package://arm_bot/meshes/body20.STL" scale="0.001 0.001 0.001"/>
       </geometry>
       <material name="">
@@ -202,5 +202,5 @@
       <origin rpy="0 1.5707 0" xyz="0.005 0 0"/>
       <geometry>
-        <mesh filename="file:///home/linux/arm_ws/src/arm_bot/meshes/body20.STL" scale="0.001 0.001 0.001"/>
+        <mesh filename="package://arm_bot/meshes/body20.STL" scale="0.001 0.001 0.001"/>
       </geometry>
     </collision>
@@ -218,5 +218,5 @@
       <origin rpy="1.5707 0.785 -1.5707" xyz="0 0 0"/>
       <geometry>
-        <mesh filename="file:///home/linux/arm_ws/src/arm_bot/meshes/Ring48_20p.STL" scale="0.001 0.001 0.001"/>
+        <mesh filename="package://arm_bot/meshes/Ring48_20p.STL" scale="0.001 0.001 0.001"/>
       </geometry>
       <material name="">
@@ -227,5 +227,5 @@
       <origin rpy="1.5707 0.785 -1.5707" xyz="0 0 0"/>
       <geometry>
-        <mesh filename="file:///home/linux/arm_ws/src/arm_bot/meshes/Ring48_20p.STL" scale="0.001 0.001 0.001"/>
+        <mesh filename="package://arm_bot/meshes/Ring48_20p.STL" scale="0.001 0.001 0.001"/>
       </geometry>
     </collision>
@@ -241,5 +241,5 @@
       <origin rpy="3.14 0 -1.5707" xyz="0.142 0 0.09525"/>
       <geometry>
-        <mesh filename="file:///home/linux/arm_ws/src/arm_bot/meshes/UpperArm.STL" scale="0.001 0.001 0.001"/>
+        <mesh filename="package://arm_bot/meshes/UpperArm.STL" scale="0.001 0.001 0.001"/>
       </geometry>
       <material name="">
@@ -250,5 +250,5 @@
       <origin rpy="3.14 0 -1.5707" xyz="0.142 0 0.09525"/>
       <geometry>
-        <mesh filename="file:///home/linux/arm_ws/src/arm_bot/meshes/UpperArm.STL" scale="0.001 0.001 0.001"/>
+        <mesh filename="package://arm_bot/meshes/UpperArm.STL" scale="0.001 0.001 0.001"/>
       </geometry>
     </collision>
@@ -264,5 +264,5 @@
       <origin rpy="0 -1.5707 3.14" xyz="-0.03655 0 0"/>
       <geometry>
-        <mesh filename="file:///home/linux/arm_ws/src/arm_bot/meshes/elbowshell.STL" scale="0.001 0.001 0.001"/>
+        <mesh filename="package://arm_bot/meshes/elbowshell.STL" scale="0.001 0.001 0.001"/>
       </geometry>
       <material name="">
@@ -273,5 +273,5 @@
       <origin rpy="0 -1.5707 3.14" xyz="-0.03655 0 0"/>
       <geometry>
-        <mesh filename="file:///home/linux/arm_ws/src/arm_bot/meshes/elbowshell.STL" scale="0.001 0.001 0.001"/>
+        <mesh filename="package://arm_bot/meshes/elbowshell.STL" scale="0.001 0.001 0.001"/>
       </geometry>
     </collision>
@@ -287,5 +287,5 @@
       <origin rpy="0 -1.5707 0" xyz="0.022 0 0"/>
       <geometry>
-        <mesh filename="file:///home/linux/arm_ws/src/arm_bot/meshes/elbowcap.STL" scale="0.001 0.001 0.001"/>
+        <mesh filename="package://arm_bot/meshes/elbowcap.STL" scale="0.001 0.001 0.001"/>
       </geometry>
       <material name="">
@@ -296,5 +296,5 @@
       <origin rpy="0 -1.5707 0" xyz="0.022 0 0"/>
       <geometry>
-        <mesh filename="file:///home/linux/arm_ws/src/arm_bot/meshes/elbowcap.STL" scale="0.001 0.001 0.001"/>
+        <mesh filename="package://arm_bot/meshes/elbowcap.STL" scale="0.001 0.001 0.001"/>
       </geometry>
     </collision>
@@ -310,5 +310,5 @@
       <origin rpy="0 -1.5707 0" xyz="0 0 0"/>
       <geometry>
-        <mesh filename="file:///home/linux/arm_ws/src/arm_bot/meshes/bodyH30_base.STL" scale="0.001 0.001 0.001"/>
+        <mesh filename="package://arm_bot/meshes/bodyH30_base.STL" scale="0.001 0.001 0.001"/>
       </geometry>
       <material name="">
@@ -319,5 +319,5 @@
       <origin rpy="0 -1.5707 0" xyz="0 0 0"/>
       <geometry>
-        <mesh filename="file:///home/linux/arm_ws/src/arm_bot/meshes/bodyH30_base.STL" scale="0.001 0.001 0.001"/>
+        <mesh filename="package://arm_bot/meshes/bodyH30_base.STL" scale="0.001 0.001 0.001"/>
       </geometry>
     </collision>
@@ -333,5 +333,5 @@
       <origin rpy="0 -1.5707 0" xyz="0 0 0"/>
       <geometry>
-        <mesh filename="file:///home/linux/arm_ws/src/arm_bot/meshes/bodyH30.STL" scale="0.001 0.001 0.001"/>
+        <mesh filename="package://arm_bot/meshes/bodyH30.STL" scale="0.001 0.001 0.001"/>
       </geometry>
       <material name="">
@@ -342,5 +342,5 @@
       <origin rpy="0 -1.5707 0" xyz="0 0 0"/>
       <geometry>
-        <mesh filename="file:///home/linux/arm_ws/src/arm_bot/meshes/bodyH30.STL" scale="0.001 0.001 0.001"/>
+        <mesh filename="package://arm_bot/meshes/bodyH30.STL" scale="0.001 0.001 0.001"/>
       </geometry>
     </collision>
@@ -358,5 +358,5 @@
       <origin rpy="1.5707 0.78535 1.5707" xyz="0 0 0"/>
       <geometry>
-        <mesh filename="file:///home/linux/arm_ws/src/arm_bot/meshes/Ring48H30.STL" scale="0.001 0.001 0.001"/>
+        <mesh filename="package://arm_bot/meshes/Ring48H30.STL" scale="0.001 0.001 0.001"/>
       </geometry>
       <material name="">
@@ -367,5 +367,5 @@
       <origin rpy="1.5707 0.78535 1.5707" xyz="0 0 0"/>
       <geometry>
-        <mesh filename="file:///home/linux/arm_ws/src/arm_bot/meshes/Ring48H30.STL" scale="0.001 0.001 0.001"/>
+        <mesh filename="package://arm_bot/meshes/Ring48H30.STL" scale="0.001 0.001 0.001"/>
       </geometry>
     </collision>
@@ -381,5 +381,5 @@
       <origin rpy="3.14 0 0" xyz="-0.025 0 0"/>
       <geometry>
-        <mesh filename="file:///home/linux/arm_ws/src/arm_bot/meshes/Forearm.STL" scale="0.001 0.001 0.001"/>
+        <mesh filename="package://arm_bot/meshes/Forearm.STL" scale="0.001 0.001 0.001"/>
       </geometry>
       <material name="">
@@ -390,5 +390,5 @@
       <origin rpy="3.14 0 0" xyz="-0.025 0 0"/>
       <geometry>
-        <mesh filename="file:///home/linux/arm_ws/src/arm_bot/meshes/Forearm.STL" scale="0.001 0.001 0.001"/>
+        <mesh filename="package://arm_bot/meshes/Forearm.STL" scale="0.001 0.001 0.001"/>
       </geometry>
     </collision>
@@ -404,5 +404,5 @@
       <origin rpy="-1.5707 0 1.5707" xyz="-0.013 0 0"/>
       <geometry>
-        <mesh filename="file:///home/linux/arm_ws/src/arm_bot/meshes/wristshell.STL" scale="0.001 0.001 0.001"/>
+        <mesh filename="package://arm_bot/meshes/wristshell.STL" scale="0.001 0.001 0.001"/>
       </geometry>
       <material name="">
@@ -413,5 +413,5 @@
       <origin rpy="-1.5707 0 1.5707" xyz="-0.013 0 0"/>
       <geometry>
-        <mesh filename="file:///home/linux/arm_ws/src/arm_bot/meshes/wristshell.STL" scale="0.001 0.001 0.001"/>
+        <mesh filename="package://arm_bot/meshes/wristshell.STL" scale="0.001 0.001 0.001"/>
       </geometry>
     </collision>
@@ -427,5 +427,5 @@
       <origin rpy="0 1.5707 0" xyz="0 0 0"/>
       <geometry>
-        <mesh filename="file:///home/linux/arm_ws/src/arm_bot/meshes/wristcap.STL" scale="0.001 0.001 0.001"/>
+        <mesh filename="package://arm_bot/meshes/wristcap.STL" scale="0.001 0.001 0.001"/>
       </geometry>
       <material name="">
@@ -436,5 +436,5 @@
       <origin rpy="0 1.5707 0" xyz="0 0 0"/>
       <geometry>
-        <mesh filename="file:///home/linux/arm_ws/src/arm_bot/meshes/wristcap.STL" scale="0.001 0.001 0.001"/>
+        <mesh filename="package://arm_bot/meshes/wristcap.STL" scale="0.001 0.001 0.001"/>
       </geometry>
     </collision>
@@ -450,5 +450,5 @@
       <origin rpy="0 1.5707 0" xyz="0 0 0"/>
       <geometry>
-        <mesh filename="file:///home/linux/arm_ws/src/arm_bot/meshes/bodyH40.STL" scale="0.001 0.001 0.001"/>
+        <mesh filename="package://arm_bot/meshes/bodyH40.STL" scale="0.001 0.001 0.001"/>
       </geometry>
       <material name="">
@@ -459,5 +459,5 @@
       <origin rpy="0 1.5707 0" xyz="0 0 0"/>
       <geometry>
-        <mesh filename="file:///home/linux/arm_ws/src/arm_bot/meshes/bodyH40.STL" scale="0.001 0.001 0.001"/>
+        <mesh filename="package://arm_bot/meshes/bodyH40.STL" scale="0.001 0.001 0.001"/>
       </geometry>
     </collision>
@@ -475,5 +475,5 @@
       <origin rpy="-1.5707 -0.78535 1.5707" xyz="0 0 0"/>
       <geometry>
-        <mesh filename="file:///home/linux/arm_ws/src/arm_bot/meshes/Ring48H40.STL" scale="0.001 0.001 0.001"/>
+        <mesh filename="package://arm_bot/meshes/Ring48H40.STL" scale="0.001 0.001 0.001"/>
       </geometry>
       <material name="">
@@ -484,5 +484,5 @@
       <origin rpy="-1.5707 -0.78535 1.5707" xyz="0 0 0"/>
       <geometry>
-        <mesh filename="file:///home/linux/arm_ws/src/arm_bot/meshes/Ring48H40.STL" scale="0.001 0.001 0.001"/>
+        <mesh filename="package://arm_bot/meshes/Ring48H40.STL" scale="0.001 0.001 0.001"/>
       </geometry>
     </collision>
@@ -498,5 +498,5 @@
       <origin rpy="3.14 0 -1.5707" xyz="0 0 0.012"/>
       <geometry>
-        <mesh filename="file:///home/linux/arm_ws/src/arm_bot/meshes/wristshell.STL" scale="0.001 0.001 0.001"/>
+        <mesh filename="package://arm_bot/meshes/wristshell.STL" scale="0.001 0.001 0.001"/>
       </geometry>
       <material name="">
@@ -507,5 +507,5 @@
       <origin rpy="3.14 0 -1.5707" xyz="0 0 0.012"/>
       <geometry>
-        <mesh filename="file:///home/linux/arm_ws/src/arm_bot/meshes/wristshell.STL" scale="0.001 0.001 0.001"/>
+        <mesh filename="package://arm_bot/meshes/wristshell.STL" scale="0.001 0.001 0.001"/>
       </geometry>
     </collision>
@@ -521,5 +521,5 @@
       <origin rpy="0 0 0" xyz="0 0 0"/>
       <geometry>
-        <mesh filename="file:///home/linux/arm_ws/src/arm_bot/meshes/wristcap.STL" scale="0.001 0.001 0.001"/>
+        <mesh filename="package://arm_bot/meshes/wristcap.STL" scale="0.001 0.001 0.001"/>
       </geometry>
       <material name="">
@@ -530,5 +530,5 @@
       <origin rpy="0 0 0" xyz="0 0 0"/>
       <geometry>
-        <mesh filename="file:///home/linux/arm_ws/src/arm_bot/meshes/wristcap.STL" scale="0.001 0.001 0.001"/>
+        <mesh filename="package://arm_bot/meshes/wristcap.STL" scale="0.001 0.001 0.001"/>
       </geometry>
     </collision>
@@ -545,5 +545,5 @@
       <origin rpy="0 0 0" xyz="0 0 0"/>
       <geometry>
-        <mesh filename="file:///home/linux/arm_ws/src/arm_bot/meshes/bodyH40.STL" scale="0.001 0.001 0.001"/>
+        <mesh filename="package://arm_bot/meshes/bodyH40.STL" scale="0.001 0.001 0.001"/>
       </geometry>
       <material name="">
@@ -554,5 +554,5 @@
       <origin rpy="0 0 0" xyz="0 0 0"/>
       <geometry>
-        <mesh filename="file:///home/linux/arm_ws/src/arm_bot/meshes/bodyH40.STL" scale="0.001 0.001 0.001"/>
+        <mesh filename="package://arm_bot/meshes/bodyH40.STL" scale="0.001 0.001 0.001"/>
       </geometry>
     </collision>
@@ -570,5 +570,5 @@
       <origin rpy="0 3.14 0.78535" xyz="0 0 0"/>
       <geometry>
-        <mesh filename="file:///home/linux/arm_ws/src/arm_bot/meshes/Ring48H40.STL" scale="0.001 0.001 0.001"/>
+        <mesh filename="package://arm_bot/meshes/Ring48H40.STL" scale="0.001 0.001 0.001"/>
       </geometry>
       <material name="">
@@ -579,5 +579,5 @@
       <origin rpy="0 3.14 0.78535" xyz="0 0 0"/>
       <geometry>
-        <mesh filename="file:///home/linux/arm_ws/src/arm_bot/meshes/Ring48H40.STL" scale="0.001 0.001 0.001"/>
+        <mesh filename="package://arm_bot/meshes/Ring48H40.STL" scale="0.001 0.001 0.001"/>
       </geometry>
     </collision>
@@ -593,5 +593,5 @@
       <origin rpy="-1.5707 0 1.5707" xyz="0.012 0 0"/>
       <geometry>
-        <mesh filename="file:///home/linux/arm_ws/src/arm_bot/meshes/wristshell.STL" scale="0.001 0.001 0.001"/>
+        <mesh filename="package://arm_bot/meshes/wristshell.STL" scale="0.001 0.001 0.001"/>
       </geometry>
       <material name="">
@@ -602,5 +602,5 @@
       <origin rpy="-1.5707 0 1.5707" xyz="0.012 0 0"/>
       <geometry>
-        <mesh filename="file:///home/linux/arm_ws/src/arm_bot/meshes/wristshell.STL" scale="0.001 0.001 0.001"/>
+        <mesh filename="package://arm_bot/meshes/wristshell.STL" scale="0.001 0.001 0.001"/>
       </geometry>
     </collision>
@@ -616,5 +616,5 @@
       <origin rpy="0 1.5707 0" xyz="0 0 0"/>
       <geometry>
-        <mesh filename="file:///home/linux/arm_ws/src/arm_bot/meshes/wristcap.STL" scale="0.001 0.001 0.001"/>
+        <mesh filename="package://arm_bot/meshes/wristcap.STL" scale="0.001 0.001 0.001"/>
       </geometry>
       <material name="">
@@ -625,5 +625,5 @@
       <origin rpy="0 1.5707 0" xyz="0 0 0"/>
       <geometry>
-        <mesh filename="file:///home/linux/arm_ws/src/arm_bot/meshes/wristcap.STL" scale="0.001 0.001 0.001"/>
+        <mesh filename="package://arm_bot/meshes/wristcap.STL" scale="0.001 0.001 0.001"/>
       </geometry>
     </collision>
@@ -639,5 +639,5 @@
       <origin rpy="0 1.5707 0" xyz="0 0 0"/>
       <geometry>
-        <mesh filename="file:///home/linux/arm_ws/src/arm_bot/meshes/bodyH40.STL" scale="0.001 0.001 0.001"/>
+        <mesh filename="package://arm_bot/meshes/bodyH40.STL" scale="0.001 0.001 0.001"/>
       </geometry>
       <material name="">
@@ -648,5 +648,5 @@
       <origin rpy="0 1.5707 0" xyz="0 0 0"/>
       <geometry>
-        <mesh filename="file:///home/linux/arm_ws/src/arm_bot/meshes/bodyH40.STL" scale="0.001 0.001 0.001"/>
+        <mesh filename="package://arm_bot/meshes/bodyH40.STL" scale="0.001 0.001 0.001"/>
       </geometry>
     </collision>
@@ -664,5 +664,5 @@
       <origin rpy="-1.5707 -0.78535 1.5707" xyz="0 0 0"/>
       <geometry>
-        <mesh filename="file:///home/linux/arm_ws/src/arm_bot/meshes/Ring48H40.STL" scale="0.001 0.001 0.001"/>
+        <mesh filename="package://arm_bot/meshes/Ring48H40.STL" scale="0.001 0.001 0.001"/>
       </geometry>
       <material name="">
@@ -673,5 +673,5 @@
       <origin rpy="-1.5707 -0.78535 1.5707" xyz="0 0 0"/>
       <geometry>
-        <mesh filename="file:///home/linux/arm_ws/src/arm_bot/meshes/Ring48H40.STL" scale="0.001 0.001 0.001"/>
+        <mesh filename="package://arm_bot/meshes/Ring48H40.STL" scale="0.001 0.001 0.001"/>
       </geometry>
     </collision>
@@ -687,5 +687,5 @@
       <origin rpy="1.5707 0 1.5707" xyz="0 0 0"/>
       <geometry>
-        <mesh filename="file:///home/linux/arm_ws/src/arm_bot/meshes/grip2plate.STL" scale="0.001 0.001 0.001"/>
+        <mesh filename="package://arm_bot/meshes/grip2plate.STL" scale="0.001 0.001 0.001"/>
       </geometry>
       <material name="">
@@ -696,5 +696,5 @@
       <origin rpy="1.5707 0 1.5707" xyz="0 0 0"/>
       <geometry>
-        <mesh filename="file:///home/linux/arm_ws/src/arm_bot/meshes/grip2plate.STL" scale="0.001 0.001 0.001"/>
+        <mesh filename="package://arm_bot/meshes/grip2plate.STL" scale="0.001 0.001 0.001"/>
       </geometry>
     </collision>
@@ -710,5 +710,5 @@
       <origin rpy="0 0 3.14" xyz="-0.1865 0.0304 0"/>
       <geometry>
-        <mesh filename="file:///home/linux/arm_ws/src/arm_bot/meshes/gripperbase2.STL" scale="0.001 0.001 0.001"/>
+        <mesh filename="package://arm_bot/meshes/gripperbase2.STL" scale="0.001 0.001 0.001"/>
       </geometry>
       <material name="">
@@ -719,5 +719,5 @@
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