Commit message: add moveit and correct the urdf collision primitives

File: arm_bot/description/robot.urdf.xacro (robot description, xacro)
@@ -60,7 +60,7 @@
     </visual>
     <collision>
-      <origin rpy="3.14 0 0" xyz="0 0 0.07785"/>
-      <geometry>
-        <mesh filename="package://arm_bot/meshes/basecone.STL" scale="0.001 0.001 0.001"/>
+      <origin rpy="3.14 0 0" xyz="0 0 0.04585"/>
+      <geometry>
+        <cylinder radius="0.065" length="0.13"/>
       </geometry>
     </collision>
@@ -72,5 +72,5 @@
   </joint>
   <link name="actuator1">
-    <xacro:default_inertial mass="1.0"/>
+    <xacro:default_inertial mass="0.1"/>
     <visual>
       <origin rpy="0 0 0" xyz="0 0 0"/>
@@ -82,10 +82,10 @@
       </material>
     </visual>
-    <collision>
+    <!-- <collision>
       <origin rpy="0 0 0" xyz="0 0 0"/>
       <geometry>
         <mesh filename="package://arm_bot/meshes/body20.STL" scale="0.001 0.001 0.001"/>
       </geometry>
-    </collision>
+    </collision> -->
   </link>
   <joint name="Joint_1" type="revolute">
@@ -94,8 +94,8 @@
     <child link="ring1"/>
     <axis xyz="0 0 1"/>
-    <limit effort="5" lower="-3.14" upper="3.14" velocity="10"/>
+    <limit effort="100" lower="-3.14" upper="3.14" velocity="10"/>
   </joint>
   <link name="ring1">
-    <xacro:default_inertial mass="1.0"/>
+    <xacro:default_inertial mass="0.1"/>
     <visual>
       <origin rpy="3.14 0 0.785" xyz="0 0 0.0"/>
@@ -107,10 +107,10 @@
       </material>
     </visual>
-    <collision>
+    <!-- <collision>
       <origin rpy="3.14 0 0.785" xyz="0 0 0.0"/>
       <geometry>
         <mesh filename="package://arm_bot/meshes/Ring48_20p.STL" scale="0.001 0.001 0.001"/>
       </geometry>
-    </collision>
+    </collision> -->
   </link>
   <joint name="ring1_fixed" type="fixed">
@@ -120,5 +120,5 @@
   </joint>
   <link name="actuator_2_holder">
-    <xacro:default_inertial mass="1.0"/>
+    <xacro:default_inertial mass="0.1"/>
     <visual>
       <origin rpy="0 0 3.14" xyz="0.0556 0.0253 0"/>
@@ -130,10 +130,10 @@
       </material>
     </visual>
-    <collision>
+    <!-- <collision>
       <origin rpy="0 0 3.14" xyz="0.0556 0.0253 0"/>
       <geometry>
         <mesh filename="package://arm_bot/meshes/shoulderplate.STL" scale="0.001 0.001 0.001"/>
       </geometry>
-    </collision>
+    </collision> -->
   </link>
   <joint name="actuator2_shell_fixed" type="fixed">
@@ -143,5 +143,5 @@
   </joint>
   <link name="actuator_2_shell">
-    <xacro:default_inertial mass="1.0"/>
+    <xacro:default_inertial mass="0.1"/>
     <visual>
       <origin rpy="-1.5707 0 1.5707" xyz="0 0 0.057"/>
@@ -156,5 +156,5 @@
       <origin rpy="-1.5707 0 1.5707" xyz="0 0 0.057"/>
       <geometry>
-        <mesh filename="package://arm_bot/meshes/shouldershell.STL" scale="0.001 0.001 0.001"/>
+        <cylinder radius="0.04" length="0.13"/>
       </geometry>
     </collision>
@@ -166,5 +166,5 @@
   </joint>
   <link name="actuator_2_cap">
-    <xacro:default_inertial mass="1.0"/>
+    <xacro:default_inertial mass="0.1"/>
     <visual>
       <origin rpy="0 1.5707 0" xyz="-0.062 0 0"/>
@@ -176,10 +176,10 @@
       </material>
     </visual>
-    <collision>
+    <!-- <collision>
       <origin rpy="0 1.5707 0" xyz="-0.062 0 0"/>
       <geometry>
         <mesh filename="package://arm_bot/meshes/shouldercap.STL" scale="0.001 0.001 0.001"/>
       </geometry>
-    </collision>
+    </collision> -->
   </link>
   <joint name="actuator2_fixed" type="fixed">
@@ -189,5 +189,5 @@
   </joint>
   <link name="actuator2">
-    <xacro:default_inertial mass="1.0"/>
+    <xacro:default_inertial mass="0.1"/>
     <visual>
       <origin rpy="0 1.5707 0" xyz="0.005 0 0"/>
@@ -199,10 +199,10 @@
       </material>
     </visual>
-    <collision>
+    <!-- <collision>
       <origin rpy="0 1.5707 0" xyz="0.005 0 0"/>
       <geometry>
         <mesh filename="package://arm_bot/meshes/body20.STL" scale="0.001 0.001 0.001"/>
       </geometry>
-    </collision>
+    </collision> -->
   </link>
   <joint name="Joint_2" type="revolute">
@@ -211,8 +211,8 @@
     <child link="ring2"/>
     <axis xyz="1 0 0"/>
-    <limit effort="5" lower="-3.14" upper="3.14" velocity="10"/>
+    <limit effort="100" lower="-3.14" upper="3.14" velocity="10"/>
   </joint>
   <link name="ring2">
-    <xacro:default_inertial mass="1.0"/>
+    <xacro:default_inertial mass="0.1"/>
     <visual>
       <origin rpy="1.5707 0.785 -1.5707" xyz="0 0 0"/>
@@ -224,10 +224,10 @@
       </material>
     </visual>
-    <collision>
+    <!-- <collision>
       <origin rpy="1.5707 0.785 -1.5707" xyz="0 0 0"/>
       <geometry>
         <mesh filename="package://arm_bot/meshes/Ring48_20p.STL" scale="0.001 0.001 0.001"/>
       </geometry>
-    </collision>
+    </collision> -->
   </link>
   <joint name="upper_arm_fixed" type="fixed">
@@ -237,5 +237,5 @@
   </joint>
   <link name="upper_arm">
-    <xacro:default_inertial mass="1.0"/>
+    <xacro:default_inertial mass="0.1"/>
     <visual>
       <origin rpy="3.14 0 -1.5707" xyz="0.142 0 0.09525"/>
@@ -248,7 +248,7 @@
     </visual>
     <collision>
-      <origin rpy="3.14 0 -1.5707" xyz="0.142 0 0.09525"/>
-      <geometry>
-        <mesh filename="package://arm_bot/meshes/UpperArm.STL" scale="0.001 0.001 0.001"/>
+      <origin rpy="3.14 0 -1.5707" xyz="0.0055 0 0.09525"/>
+      <geometry>
+        <cylinder radius="0.025" length="0.17"/>
       </geometry>
     </collision>
@@ -260,5 +260,5 @@
   </joint>
   <link name="elbow_shell">
-    <xacro:default_inertial mass="1.0"/>
+    <xacro:default_inertial mass="0.1"/>
     <visual>
       <origin rpy="0 -1.5707 3.14" xyz="-0.03655 0 0"/>
@@ -273,5 +273,5 @@
       <origin rpy="0 -1.5707 3.14" xyz="-0.03655 0 0"/>
       <geometry>
-        <mesh filename="package://arm_bot/meshes/elbowshell.STL" scale="0.001 0.001 0.001"/>
+        <cylinder radius="0.03" length="0.13"/>
       </geometry>
     </collision>
@@ -283,5 +283,5 @@
   </joint>
   <link name="elbow_cap">
-    <xacro:default_inertial mass="1.0"/>
+    <xacro:default_inertial mass="0.1"/>
     <visual>
       <origin rpy="0 -1.5707 0" xyz="0.022 0 0"/>
@@ -293,10 +293,10 @@
       </material>
     </visual>
-    <collision>
+    <!-- <collision>
       <origin rpy="0 -1.5707 0" xyz="0.022 0 0"/>
       <geometry>
         <mesh filename="package://arm_bot/meshes/elbowcap.STL" scale="0.001 0.001 0.001"/>
       </geometry>
-    </collision>
+    </collision> -->
   </link>
   <joint name="actuator3_base_fixed" type="fixed">
@@ -306,5 +306,5 @@
   </joint>
   <link name="actuator3_base">
-    <xacro:default_inertial mass="1.0"/>
+    <xacro:default_inertial mass="0.1"/>
     <visual>
       <origin rpy="0 -1.5707 0" xyz="0 0 0"/>
@@ -316,10 +316,10 @@
       </material>
     </visual>
-    <collision>
+    <!-- <collision>
       <origin rpy="0 -1.5707 0" xyz="0 0 0"/>
       <geometry>
         <mesh filename="package://arm_bot/meshes/bodyH30_base.STL" scale="0.001 0.001 0.001"/>
       </geometry>
-    </collision>
+    </collision> -->
   </link>
   <joint name="actuator3_fixed" type="fixed">
@@ -329,5 +329,5 @@
   </joint>
   <link name="actuator3">
-    <xacro:default_inertial mass="1.0"/>
+    <xacro:default_inertial mass="0.1"/>
     <visual>
       <origin rpy="0 -1.5707 0" xyz="0 0 0"/>
@@ -339,10 +339,10 @@
       </material>
     </visual>
-    <collision>
+    <!-- <collision>
       <origin rpy="0 -1.5707 0" xyz="0 0 0"/>
       <geometry>
         <mesh filename="package://arm_bot/meshes/bodyH30.STL" scale="0.001 0.001 0.001"/>
       </geometry>
-    </collision>
+    </collision> -->
   </link>
   <joint name="Joint_3" type="revolute">
@@ -351,8 +351,8 @@
     <child link="ring3"/>
     <axis xyz="1 0 0"/>
-    <limit effort="5" lower="-3.14" upper="3.14" velocity="10"/>
+    <limit effort="100" lower="-3.14" upper="3.14" velocity="10"/>
   </joint>
   <link name="ring3">
-    <xacro:default_inertial mass="1.0"/>
+    <xacro:default_inertial mass="0.1"/>
     <visual>
       <origin rpy="1.5707 0.78535 1.5707" xyz="0 0 0"/>
@@ -364,10 +364,10 @@
       </material>
     </visual>
-    <collision>
+    <!-- <collision>
       <origin rpy="1.5707 0.78535 1.5707" xyz="0 0 0"/>
       <geometry>
         <mesh filename="package://arm_bot/meshes/Ring48H30.STL" scale="0.001 0.001 0.001"/>
       </geometry>
-    </collision>
+    </collision> -->
   </link>
   <joint name="fore_arm_fixed" type="fixed">
@@ -377,5 +377,5 @@
   </joint>
   <link name="fore_arm">
-    <xacro:default_inertial mass="1.0"/>
+    <xacro:default_inertial mass="0.1"/>
     <visual>
       <origin rpy="3.14 0 0" xyz="-0.025 0 0"/>
@@ -388,7 +388,7 @@
     </visual>
     <collision>
-      <origin rpy="3.14 0 0" xyz="-0.025 0 0"/>
-      <geometry>
-        <mesh filename="package://arm_bot/meshes/Forearm.STL" scale="0.001 0.001 0.001"/>
+      <origin rpy="3.14 0 0" xyz="-0.025 0 -0.085"/>
+      <geometry>
+        <cylinder radius="0.02" length="0.17"/>
       </geometry>
     </collision>
@@ -400,5 +400,5 @@
   </joint>
   <link name="actuator4_shell">
-    <xacro:default_inertial mass="1.0"/>
+    <xacro:default_inertial mass="0.1"/>
     <visual>
       <origin rpy="-1.5707 0 1.5707" xyz="-0.013 0 0"/>
@@ -411,7 +411,7 @@
     </visual>
     <collision>
-      <origin rpy="-1.5707 0 1.5707" xyz="-0.013 0 0"/>
-      <geometry>
-        <mesh filename="package://arm_bot/meshes/wristshell.STL" scale="0.001 0.001 0.001"/>
+      <origin rpy="-1.5707 0 1.5707" xyz="-0.021 0 0"/>
+      <geometry>
+        <cylinder radius="0.03" length="0.06"/>
       </geometry>
     </collision>
@@ -423,5 +423,5 @@
   </joint>
   <link name="actuator4_cap">
-    <xacro:default_inertial mass="1.0"/>
+    <xacro:default_inertial mass="0.1"/>
     <visual>
       <origin rpy="0 1.5707 0" xyz="0 0 0"/>
@@ -433,10 +433,10 @@
       </material>
     </visual>
-    <collision>
+    <!-- <collision>
       <origin rpy="0 1.5707 0" xyz="0 0 0"/>
       <geometry>
         <mesh filename="package://arm_bot/meshes/wristcap.STL" scale="0.001 0.001 0.001"/>
       </geometry>
-    </collision>
+    </collision> -->
   </link>
   <joint name="actuator4_fixed" type="fixed">
@@ -446,5 +446,5 @@
   </joint>
   <link name="actuator4">
-    <xacro:default_inertial mass="1.0"/>
+    <xacro:default_inertial mass="0.1"/>
     <visual>
       <origin rpy="0 1.5707 0" xyz="0 0 0"/>
@@ -456,10 +456,10 @@
       </material>
     </visual>
-    <collision>
+    <!-- <collision>
       <origin rpy="0 1.5707 0" xyz="0 0 0"/>
       <geometry>
         <mesh filename="package://arm_bot/meshes/bodyH40.STL" scale="0.001 0.001 0.001"/>
       </geometry>
-    </collision>
+    </collision> -->
   </link>
   <joint name="Joint_4" type="revolute">
@@ -468,8 +468,8 @@
     <child link="ring4"/>
     <axis xyz="1 0 0"/>
-    <limit effort="5" lower="-3.14" upper="3.14" velocity="10"/>
+    <limit effort="100" lower="-3.14" upper="3.14" velocity="10"/>
   </joint>
   <link name="ring4">
-    <xacro:default_inertial mass="1.0"/>
+    <xacro:default_inertial mass="0.1"/>
     <visual>
       <origin rpy="-1.5707 -0.78535 1.5707" xyz="0 0 0"/>
@@ -481,10 +481,10 @@
       </material>
     </visual>
-    <collision>
+    <!-- <collision>
       <origin rpy="-1.5707 -0.78535 1.5707" xyz="0 0 0"/>
       <geometry>
         <mesh filename="package://arm_bot/meshes/Ring48H40.STL" scale="0.001 0.001 0.001"/>
       </geometry>
-    </collision>
+    </collision> -->
   </link>
   <joint name="actuator5_shell_fixed" type="fixed">
@@ -494,5 +494,5 @@
   </joint>
   <link name="actuator5_shell">
-    <xacro:default_inertial mass="1.0"/>
+    <xacro:default_inertial mass="0.1"/>
     <visual>
       <origin rpy="3.14 0 -1.5707" xyz="0 0 0.012"/>
@@ -505,7 +505,7 @@
     </visual>
     <collision>
-      <origin rpy="3.14 0 -1.5707" xyz="0 0 0.012"/>
-      <geometry>
-        <mesh filename="package://arm_bot/meshes/wristshell.STL" scale="0.001 0.001 0.001"/>
+      <origin rpy="3.14 0 -1.5707" xyz="0 0 0.005"/>
+      <geometry>
+        <cylinder radius="0.03" length="0.06"/>
       </geometry>
     </collision>
@@ -517,5 +517,5 @@
   </joint>
   <link name="actuator5_cap">
-    <xacro:default_inertial mass="1.0"/>
+    <xacro:default_inertial mass="0.1"/>
     <visual>
       <origin rpy="0 0 0" xyz="0 0 0"/>
@@ -527,10 +527,10 @@
       </material>
     </visual>
-    <collision>
+    <!-- <collision>
       <origin rpy="0 0 0" xyz="0 0 0"/>
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